Commit message: community code to ros2 jazzy migratrion

File: cobot_ws_addition/src/mycobot_ros2/mycobot_description/urdf/control/mycobot_280_ros2_control.urdf.xacro (robot description, xacro)
@@ -59,29 +59,20 @@
             </joint>
             <joint name="${prefix}gripper_base_to_${prefix}gripper_left2">
-                <param name="mimic">gripper_controller</param>
-                <param name="multiplier">1.0</param>
                 <state_interface name="position"/>
                 <state_interface name="velocity"/>
             </joint>
             <joint name="${prefix}gripper_left3_to_${prefix}gripper_left1">
-                <param name="mimic">gripper_controller</param>
-                <param name="multiplier">-1.0</param>
                 <state_interface name="position"/>
                 <state_interface name="velocity"/>
             </joint>
             <joint name="${prefix}gripper_base_to_${prefix}gripper_right3">
-                <param name="mimic">gripper_controller</param>
-                <param name="multiplier">-1.0</param>
                 <state_interface name="position"/>
                 <state_interface name="velocity"/>
             </joint>
             <joint name="${prefix}gripper_base_to_${prefix}gripper_right2">
-                <param name="mimic">gripper_controller</param>
                 <state_interface name="position"/>
                 <state_interface name="velocity"/>
             </joint>
             <joint name="${prefix}gripper_right3_to_${prefix}gripper_right1">
-                <param name="mimic">gripper_controller</param>
-                <param name="multiplier">1.0</param>
                 <state_interface name="position"/>
                 <state_interface name="velocity"/>

File: cobot_ws_addition/src/mycobot_ros2/mycobot_description/urdf/mech/adaptive_gripper.urdf.xacro (robot description, xacro)
@@ -151,5 +151,4 @@
       <child link="${prefix}gripper_left2"/>
       <origin xyz="-0.005 0.027 0" rpy="0 0 0"/>
-      <mimic joint="${prefix}gripper_controller" multiplier="1.0" offset="0"/>
       <dynamics damping="${joint_damping}" friction="${joint_friction}"/>
     </joint>
@@ -160,5 +159,4 @@
       <child link="${prefix}gripper_left1"/>
       <origin xyz="-0.027 0.016 0" rpy="0 0 0"/>
-      <mimic joint="${prefix}gripper_controller" multiplier="-1.0" offset="0"/>
       <dynamics damping="${joint_damping}" friction="${joint_friction}"/>
     </joint>
@@ -169,5 +167,4 @@
       <child link="${prefix}gripper_right3"/>
       <origin xyz="0.012 0.005 0" rpy="0 0 0"/>
-      <mimic joint="${prefix}gripper_controller" multiplier="-1.0" offset="0"/>
       <dynamics damping="${joint_damping}" friction="${joint_friction}"/>
     </joint>
@@ -178,5 +175,4 @@
       <child link="${prefix}gripper_right2"/>
       <origin xyz="0.005 0.027 0" rpy="0 0 0"/>
-      <mimic joint="${prefix}gripper_controller" multiplier="-1.0" offset="0"/>
       <dynamics damping="${joint_damping}" friction="${joint_friction}"/>
     </joint>
@@ -187,5 +183,4 @@
       <child link="${prefix}gripper_right1"/>
       <origin xyz="0.027 0.016 0" rpy="0 0 0"/>
-      <mimic joint="${prefix}gripper_controller" multiplier="1.0" offset="0"/>
       <dynamics damping="${joint_damping}" friction="${joint_friction}"/>
     </joint>
